File: hardware/logicboard/midiext-led-001.brd (EAGLE design)
At the start: 12.7 x 25.4 mm, 4 parts, among them J1 LED

Commit message: Fixed values.
Other:
- board text added: "+"
Changed lines of the file:
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@@
 <hole x="5.08" y="2.54" drill="1.99898125"/>
 <hole x="5.08" y="22.86" drill="1.99898125"/>
+<text x="10.16" y="17.78" size="1.778" layer="1">+</text>
 </plain>
 <attributes>
