File: hardware/logicboard/longranger-001.brd (EAGLE design)
At the start: 23.5 x 72 mm, 23 parts, among them IC1 74LS07N, IC2 LTC485N, IC3 LTC485N

Commit message: Changed signal name.
Connections:
- net N$1 renamed COM1
- net N$4 renamed INDICATOR
- net N$6 renamed MUTE
Changed lines of the file:
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@@
 </class>
 </classes>
-<designrules name="pban_5mil-l2">
+<designrules name="pban_5mil-l2 *">
 <description language="de">&lt;b&gt;EAGLE Design Rules&lt;/b&gt;
 &lt;p&gt;
@@
 <param name="mtCopper" value="0.035mm 0.035mm 0.035mm 0.035mm 0.035mm 0.035mm 0.035mm 0.035mm 0.035mm 0.035mm 0.035mm 0.035mm 0.035mm 0.035mm 0.035mm 0.035mm"/>
 <param name="mtIsolate" value="1.53mm 1.5mm 0.2mm 0.15mm 0.2mm 0.15mm 0.2mm 0.15mm 0.2mm 0.15mm 0.2mm 0.15mm 0.2mm 0.15mm 0.2mm"/>
-<param name="mdWireWire" value="5mil"/>
-<param name="mdWirePad" value="0.229mm"/>
-<param name="mdWireVia" value="0.229mm"/>
-<param name="mdPadPad" value="5mil"/>
-<param name="mdPadVia" value="0.229mm"/>
-<param name="mdViaVia" value="5mil"/>
+<param name="mdWireWire" value="10mil"/>
+<param name="mdWirePad" value="10mil"/>
+<param name="mdWireVia" value="10mil"/>
+<param name="mdPadPad" value="10mil"/>
+<param name="mdPadVia" value="10mil"/>
+<param name="mdViaVia" value="10mil"/>
 <param name="mdSmdPad" value="5mil"/>
 <param name="mdSmdVia" value="5mil"/>
@@
 <wire x1="17.272" y1="64.008" x2="17.5" y2="64" width="0.254" layer="1"/>
 </signal>
-<signal name="N$1">
+<signal name="COM1">
 <contactref element="IC2" pad="1"/>
 <contactref element="IC1" pad="1"/>
@@
 <wire x1="2.54" y1="31.75" x2="4.318" y2="29.972" width="0.254" layer="16"/>
 </signal>
-<signal name="N$4">
+<signal name="INDICATOR">
 <contactref element="FRONT" pad="3"/>
 <contactref element="R5" pad="1"/>
@@
 <wire x1="6.096" y1="18.034" x2="6" y2="18" width="0.254" layer="16"/>
 </signal>
-<signal name="N$6">
+<signal name="MUTE">
 <contactref element="IC3" pad="3"/>
 <contactref element="R4" pad="2"/>
